File: hardware/Electrical/SensorArduinoHat/SensorArduinoHat.kicad_sch (KiCad schematic)
At the start: 32 parts, among them J1 Power, J2 Digital/PWM, J3 Analog, J4 Digital/PWM, U1 SN74AHC86N, U6 CD4050BE, U7 CD74HC14E

Commit message: updated readme, and fixed library linking for the arduino hat board
Parts:
- U1: footprint SN74AHC86N:N14 -> N14
- U6: footprint CD4050BE:N16 -> N16
- U7: footprint CD74HC14E:N14 -> N14
Changed lines of the file:
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@@
       (effects (font (size 1.524 1.524)))
     )
-    (property "Footprint" "CD74HC14E:N14" (at 87.63 43.18 0)
+    (property "Footprint" "N14" (at 87.63 43.18 0)
       (effects (font (size 1.27 1.27) italic) hide)
     )
@@
       (effects (font (size 1.524 1.524)))
     )
-    (property "Footprint" "CD4050BE:N16" (at 74.93 87.63 0)
+    (property "Footprint" "N16" (at 74.93 87.63 0)
       (effects (font (size 1.27 1.27) italic) hide)
     )
@@
       (effects (font (size 1.524 1.524)))
     )
-    (property "Footprint" "SN74AHC86N:N14" (at 180.34 27.94 0)
+    (property "Footprint" "N14" (at 180.34 27.94 0)
       (effects (font (size 1.27 1.27) italic) hide)
     )
